File: Eagle/psb schematic.brd (EAGLE design)
At the start: 100 x 80 mm, 12 parts, among them J1 CONN_26X2

Commit message: Correzioni PCB
Parts:
- removed J2, J3: (no value), SparkFun-Connectors:1X07
- removed R2, R3, R4: 2.0k, SparkFun-Resistors:0603
- added D1: RED, SparkFun-LED:LED-0603
- added ON/OFF: MOMENTARY-SWITCH-SPST-SMD-6.0X3.5MM, SparkFun-Switches:TACTILE_SWITCH_SMD_6.0X3.5MM
- added PIN_10: (no value), SparkFun-Connectors:1X01
- added PIN_123-124, PSOC_AL: (no value), SparkFun-Connectors:1X02
- added PIN_26-24: (no value), SparkFun-Connectors:1X04
- added R5, R6, R7, R8: (no value), SparkFun-Resistors:AXIAL-0.3
- BLUETOOTH: device SparkFun-Connectors:1X04 -> SparkFun-Connectors:1X02
- J1: value CONN_26X2 -> (none); device SparkFun-Connectors:2X26 -> SparkFun-Connectors:1X02
- R1: value 2.0k -> (none); device SparkFun-Resistors:0603 -> SparkFun-Resistors:AXIAL-0.3
- moved J1 49.4 mm to (19.1, 50.8), turned to 270 degrees
- moved R1 47.6 mm to (33.0, 45.7)
- moved FLEX1 42.4 mm to (43.2, 47.0), turned to 0 degrees
- moved FLEX2 38.1 mm to (58.4, 47.0), turned to 0 degrees
- moved FLEX3 35.4 mm to (71.1, 47.0)
- moved FSR 32.4 mm to (81.3, 45.7)
- moved BLUETOOTH 23.9 mm to (52.1, 33.0), turned to 180 degrees
Connections:
- removed net N$7: BLUETOOTH.3, J1.16
- removed net N$8: BLUETOOTH.4, J1.18
- new net N$10: D1.A, PIN_10.1
- new net N$11: D1.C, R1.P$2
- new net N$9: FLEX1.1, FLEX2.1, FLEX3.1, FSR.1, ON/OFF.1, PSOC_AL.2
- net 5V: now also J1.1, ON/OFF.2; no longer FLEX1.1, FLEX2.1, FLEX3.1, FSR.1, J1.2
- net GND: now also J1.2, PSOC_AL.1, R1.P$1, R5.P$2, R6.P$2, R7.P$2, R8.P$2; no longer J1.4, R1.1, R2.1, R3.2, R4.1
- net N$1: now also PIN_26-24.4, R5.P$1; no longer J1.42, R1.2
- net N$2: now also FLEX2.2, PIN_26-24.3, R6.P$1; no longer FSR.2, J1.48, R4.2
- net N$3: now also FLEX3.2, PIN_26-24.2, R7.P$1; no longer FLEX2.2, J1.44, R2.2
- net N$4: now also PIN_123-124.2; no longer J1.12
- net N$5: now also FSR.2, PIN_26-24.1, R8.P$1; no longer FLEX3.2, J1.46, R3.1
- net N$6: now also PIN_123-124.1; no longer J1.14
